Commit message: Added the car model

File: lane_painting_path_robot/urdf/robot.urdf.xacro (robot description, xacro)
@@ -2,12 +2,12 @@
 <robot name="lane_following_robot" xmlns:xacro="http://www.ros.org/wiki/xacro">
   <!-- Robot Properties -->
-  <xacro:property name="base_width" value="0.3"/>
-  <xacro:property name="base_length" value="0.4"/>
-  <xacro:property name="base_height" value="0.15"/>
-  <xacro:property name="wheel_radius" value="0.1"/>
-  <xacro:property name="wheel_width" value="0.05"/>
-  <xacro:property name="wheel_separation" value="0.3"/>
-  <xacro:property name="camera_size" value="0.05"/>
-  <!-- Base Link -->
+  <xacro:property name="base_width" value="0.6"/>
+  <xacro:property name="base_length" value="0.8"/>
+  <xacro:property name="base_height" value="0.3"/>
+  <xacro:property name="wheel_radius" value="0.15"/>
+  <xacro:property name="wheel_width" value="0.1"/>
+  <xacro:property name="wheel_separation" value="0.5"/>
+  <xacro:property name="camera_size" value="0.1"/>
+  <!-- Base Link (Car Body) -->
   <link name="base_link">
     <visual>
@@ -15,6 +15,6 @@
         <box size="${base_length} ${base_width} ${base_height}"/>
       </geometry>
-      <material name="blue">
-        <color rgba="0 0 1 1"/>
+      <material name="metallic_blue">
+        <color rgba="0.1 0.3 0.8 1"/>
       </material>
     </visual>
@@ -25,5 +25,27 @@
     </collision>
     <inertial>
-      <mass value="5.0"/>
+      <mass value="10.0"/>
+      <origin xyz="0 0 0" rpy="0 0 0"/>
+      <inertia ixx="0.4" ixy="0" ixz="0" iyy="0.4" iyz="0" izz="0.7"/>
+    </inertial>
+  </link>
+  <!-- Car Hood -->
+  <link name="hood_link">
+    <visual>
+      <geometry>
+        <box size="${base_length/2} ${base_width*0.9} ${base_height/2}"/>
+      </geometry>
+      <material name="metallic_blue">
+        <color rgba="0.1 0.3 0.8 1"/>
+      </material>
+    </visual>
+    <collision>
+      <geometry>
+        <box size="${base_length/2} ${base_width*0.9} ${base_height/2}"/>
+      </geometry>
+    </collision>
+    <inertial>
+      <mass value="2.0"/>
+      <origin xyz="0 0 0" rpy="0 0 0"/>
       <inertia ixx="0.1" ixy="0" ixz="0" iyy="0.1" iyz="0" izz="0.1"/>
     </inertial>
@@ -35,4 +57,46 @@
         <cylinder radius="${wheel_radius}" length="${wheel_width}"/>
       </geometry>
+      <material name="dark_gray">
+        <color rgba="0.2 0.2 0.2 1"/>
+      </material>
+    </visual>
+    <collision>
+      <geometry>
+        <cylinder radius="${wheel_radius}" length="${wheel_width}"/>
+      </geometry>
+    </collision>
+    <inertial>
+      <mass value="2.0"/>
+      <origin xyz="0 0 0" rpy="0 0 0"/>
+      <inertia ixx="0.1" ixy="0" ixz="0" iyy="0.1" iyz="0" izz="0.1"/>
+    </inertial>
+  </link>
+  <!-- Right Wheel -->
+  <link name="right_wheel">
+    <visual>
+      <geometry>
+        <cylinder radius="${wheel_radius}" length="${wheel_width}"/>
+      </geometry>
+      <material name="dark_gray">
+        <color rgba="0.2 0.2 0.2 1"/>
+      </material>
+    </visual>
+    <collision>
+      <geometry>
+        <cylinder radius="${wheel_radius}" length="${wheel_width}"/>
+      </geometry>
+    </collision>
+    <inertial>
+      <mass value="2.0"/>
+      <origin xyz="0 0 0" rpy="0 0 0"/>
+      <inertia ixx="0.1" ixy="0" ixz="0" iyy="0.1" iyz="0" izz="0.1"/>
+    </inertial>
+  </link>
+  <!-- Camera Link -->
+  <link name="camera_link">
+    <visual>
+      <geometry>
+        <box size="${camera_size} ${camera_size*2} ${camera_size}"/>
+      </geometry>
       <material name="black">
         <color rgba="0 0 0 1"/>
@@ -41,69 +105,37 @@
     <collision>
       <geometry>
-        <cylinder radius="${wheel_radius}" length="${wheel_width}"/>
-      </geometry>
-    </collision>
-    <inertial>
-      <mass value="1.0"/>
-      <inertia ixx="0.1" ixy="0" ixz="0" iyy="0.1" iyz="0" izz="0.1"/>
-    </inertial>
-  </link>
-  <!-- Right Wheel -->
-  <link name="right_wheel">
-    <visual>
-      <geometry>
-        <cylinder radius="${wheel_radius}" length="${wheel_width}"/>
-      </geometry>
-      <material name="black">
-        <color rgba="0 0 0 1"/>
-      </material>
-    </visual>
-    <collision>
-      <geometry>
-        <cylinder radius="${wheel_radius}" length="${wheel_width}"/>
-      </geometry>
-    </collision>
-    <inertial>
-      <mass value="1.0"/>
-      <inertia ixx="0.1" ixy="0" ixz="0" iyy="0.1" iyz="0" izz="0.1"/>
-    </inertial>
-  </link>
-  <!-- Camera Link -->
-  <link name="camera_link">
-    <visual>
-      <geometry>
-        <box size="${camera_size} ${camera_size} ${camera_size}"/>
-      </geometry>
-      <material name="red">
-        <color rgba="1 0 0 1"/>
-      </material>
-    </visual>
-    <collision>
-      <geometry>
-        <box size="${camera_size} ${camera_size} ${camera_size}"/>
+        <box size="${camera_size} ${camera_size*2} ${camera_size}"/>
       </geometry>
     </collision>
     <inertial>
       <mass value="0.1"/>
-      <inertia ixx="0.1" ixy="0" ixz="0" iyy="0.1" iyz="0" izz="0.1"/>
+      <origin xyz="0 0 0" rpy="0 0 0"/>
+      <inertia ixx="0.0001" ixy="0" ixz="0" iyy="0.0001" iyz="0" izz="0.0001"/>
     </inertial>
   </link>
   <!-- Joints -->
+  <joint name="hood_joint" type="fixed">
+    <parent link="base_link"/>
+    <child link="hood_link"/>
+    <origin xyz="${base_length/4} 0 ${base_height/2}" rpy="0 0 0"/>
+  </joint>
   <joint name="left_wheel_joint" type="continuous">
     <parent link="base_link"/>
     <child link="left_wheel"/>
-    <origin xyz="0 ${wheel_separation/2} 0" rpy="${pi/2} 0 0"/>
+    <origin xyz="0 ${wheel_separation/2} -0.05" rpy="${pi/2} 0 0"/>
     <axis xyz="0 0 1"/>
+    <dynamics damping="0.1" friction="0.1"/>
   </joint>
   <joint name="right_wheel_joint" type="continuous">
     <parent link="base_link"/>
     <child link="right_wheel"/>
-    <origin xyz="0 ${-wheel_separation/2} 0" rpy="${pi/2} 0 0"/>
+    <origin xyz="0 ${-wheel_separation/2} -0.05" rpy="${pi/2} 0 0"/>
     <axis xyz="0 0 1"/>
+    <dynamics damping="0.1" friction="0.1"/>
   </joint>
   <joint name="camera_joint" type="fixed">
-    <parent link="base_link"/>
+    <parent link="hood_link"/>
     <child link="camera_link"/>
-    <origin xyz="${base_length/2} 0 ${base_height/2}" rpy="0 0.3 0"/>
+    <origin xyz="${base_length/4} 0 ${base_height/4}" rpy="0 0.3 0"/>
   </joint>
   <!-- Gazebo plugins -->
@@ -115,5 +147,11 @@
       <wheel_separation>${wheel_separation}</wheel_separation>
       <wheel_radius>${wheel_radius}</wheel_radius>
-      <odom_publish_frequency>10</odom_publish_frequency>
+      <odom_publish_frequency>20</odom_publish_frequency>
+      <max_linear_velocity>2.0</max_linear_velocity>
+      <min_linear_velocity>-2.0</min_linear_velocity>
+      <max_angular_velocity>2.0</max_angular_velocity>
+      <min_angular_velocity>-2.0</min_angular_velocity>
+      <max_linear_acceleration>1.0</max_linear_acceleration>
+      <max_angular_acceleration>2.0</max_angular_acceleration>
       <topic>cmd_vel</topic>
     </plugin>
@@ -124,8 +162,8 @@
       <update_rate>30.0</update_rate>
       <camera name="head">
-        <horizontal_fov>1.3962634</horizontal_fov>
+        <horizontal_fov>1.0472</horizontal_fov>
         <image>
-          <width>800</width>
-          <height>600</height>
+          <width>640</width>
+          <height>480</height>
           <format>R8G8B8</format>
         </image>
@@ -134,4 +172,9 @@
           <far>300</far>
         </clip>
+        <noise>
+          <type>gaussian</type>
+          <mean>0.0</mean>
+          <stddev>0.007</stddev>
+        </noise>
       </camera>
       <plugin filename="gz-sim-camera-system"
@@ -142,3 +185,51 @@
     </sensor>
   </gazebo>
+  <!-- Material colors for Gazebo -->
+  <gazebo reference="base_link">
+    <material>Gazebo/Blue</material>
+    <visual>
+      <material>
+        <ambient>0.1 0.3 0.8 1</ambient>
+        <diffuse>0.1 0.3 0.8 1</diffuse>
+        <specular>0.5 0.5 0.5 1</specular>
+      </material>
+    </visual>
+  </gazebo>
+  <gazebo reference="hood_link">
+    <material>Gazebo/Blue</material>
+    <visual>
+      <material>
+        <ambient>0.1 0.3 0.8 1</ambient>
+        <diffuse>0.1 0.3 0.8 1</diffuse>
+        <specular>0.5 0.5 0.5 1</specular>
+      </material>
+    </visual>
+  </gazebo>
+  <gazebo reference="left_wheel">
+    <material>Gazebo/DarkGrey</material>
+    <mu1>1.0</mu1>
+    <mu2>1.0</mu2>
+    <visual>
+      <material>
+        <ambient>0.2 0.2 0.2 1</ambient>
+        <diffuse>0.2 0.2 0.2 1</diffuse>
+        <specular>0.5 0.5 0.5 1</specular>
+      </material>
+    </visual>
+  </gazebo>
+  <gazebo reference="right_wheel">
+    <material>Gazebo/DarkGrey</material>
+    <mu1>1.0</mu1>
+    <mu2>1.0</mu2>
+    <visual>
+      <material>
+        <ambient>0.2 0.2 0.2 1</ambient>
+        <diffuse>0.2 0.2 0.2 1</diffuse>
+        <specular>0.5 0.5 0.5 1</specular>
+      </material>
+    </visual>
+  </gazebo>
+  <gazebo reference="camera_link">
+    <material>Gazebo/Black</material>
+  </gazebo>
 </robot>
